File: sdr.kicad_pcb (KiCad board)
At the start: 4 copper layers, 65 x 30 mm, 161 parts, among them J1 SMA_H, J2 SMA_H, T1 B0322J5050, T2 B0322J5050, U1 FT601, U10 MIC94310, U11 PAM2305, U2 ESD7016, U3 LMS6002DR2, U4 ECP5, U5 Si5351, U6 PAM2305, U7 NCP186, U8 MIC94310, U9 MIC94310, X1 GSB443133HR, X2 CONN_01X08, X3 RaspberryPiConnector, Y1 FL3000027, Y2 ABM11-141-26.000MHZ

Commit message: Right before switching to full RPi
Parts:
- L3: moved to F.Cu
- moved R29 23.2 mm to (75.1, 139.5)
- moved C59 22.6 mm to (71.1, 142.7)
- moved C73 22.6 mm to (79.9, 132.7)
- moved C88 22.6 mm to (80.4, 136.8)
- moved C89 22.6 mm to (79.7, 140.8)
- moved C94 22.6 mm to (75.6, 143.7)
- moved R30 22.6 mm to (70.6, 138.4)
- moved R31 22.6 mm to (75.1, 136.5)
- moved R32 22.6 mm to (70.2, 132.8)
- moved R33 22.6 mm to (75.2, 133.1)
- moved R34 22.6 mm to (70.0, 135.4)
- moved L3 5.40 mm to (117.0, 124.0), turned to 270 degrees
- moved C79 3.29 mm to (119.9, 122.3), turned to 0 degrees
- moved C78 2.75 mm to (122.3, 124.1)
Connections:
- C78 pad 1: Net-(C78-Pad1) -> LMS_D3V3
- L3 pad 1: LMS_D3V3 -> LMS_A3V3
- L3 pad 2: Net-(C78-Pad1) -> Net-(C79-Pad1)
- U7 pad 1: Net-(U7-Pad1) -> Net-(C79-Pad1)
- U7 pad 2: Net-(U7-Pad1) -> Net-(C79-Pad1)
- U7 pad 4: Net-(U7-Pad1) -> Net-(C79-Pad1)
- U7 pad 6: Net-(C78-Pad1) -> LMS_D3V3
- U7 pad 7: Net-(C78-Pad1) -> LMS_D3V3
- U7 pad 8: Net-(C78-Pad1) -> LMS_D3V3
Changed lines of the file:
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@@
 (kicad_pcb (version 4) (host pcbnew 4.0.6-e0-6349~53~ubuntu14.04.1)
   (general
-    (links 694)
-    (no_connects 269)
+    (links 696)
+    (no_connects 271)
     (area 99.924999 99.924999 165.075001 130.075001)
     (thickness 1.6)
@@
     (zones 0)
     (modules 161)
-    (nets 273)
+    (nets 271)
   )
   (page A4)
@@
     (34 B.Paste user hide)
     (35 F.Paste user hide)
-    (36 B.SilkS user hide)
-    (37 F.SilkS user hide)
+    (36 B.SilkS user)
+    (37 F.SilkS user)
     (38 B.Mask user hide)
     (39 F.Mask user hide)
@@
     (pad_to_mask_clearance 0.2)
     (aux_axis_origin 124.58 122.04)
-    (visible_elements FFFEFF7F)
+    (visible_elements FFFEF77F)
     (pcbplotparams
       (layerselection 0x00030_80000001)
@@
   (net 269 "Net-(L8-Pad2)")
   (net 270 "Net-(L9-Pad2)")
-  (net 271 "Net-(C78-Pad1)")
-  (net 272 "Net-(U7-Pad1)")
   (net_class Default "This is the default net class."
     (clearance 0.127)
@@
     (add_net "Net-(C76-Pad1)")
     (add_net "Net-(C77-Pad2)")
-    (add_net "Net-(C78-Pad1)")
     (add_net "Net-(C79-Pad1)")
     (add_net "Net-(C86-Pad1)")
@@
     (add_net "Net-(U5-Pad2)")
     (add_net "Net-(U5-Pad3)")
-    (add_net "Net-(U7-Pad1)")
     (add_net "Net-(X1-PadOTG)")
     (add_net RPI_A0)
@@
     (fp_line (start -1.35 -1.125) (end 0.575 -1.125) (layer F.SilkS) (width 0.15))
     (pad 1 smd rect (at -0.65 -0.6) (size 0.5 0.25) (layers F.Cu F.Paste F.Mask)
-      (net 272 "Net-(U7-Pad1)"))
+      (net 247 "Net-(C79-Pad1)"))
     (pad 2 smd rect (at -0.65 -0.2) (size 0.5 0.25) (layers F.Cu F.Paste F.Mask)
-      (net 272 "Net-(U7-Pad1)"))
+      (net 247 "Net-(C79-Pad1)"))
     (pad 3 smd rect (at -0.65 0.2) (size 0.5 0.25) (layers F.Cu F.Paste F.Mask)
       (net 3 GNDD))
     (pad 4 smd rect (at -0.65 0.6) (size 0.5 0.25) (layers F.Cu F.Paste F.Mask)
-      (net 272 "Net-(U7-Pad1)"))
+      (net 247 "Net-(C79-Pad1)"))
     (pad 5 smd rect (at 0.65 0.6) (size 0.5 0.25) (layers F.Cu F.Paste F.Mask)
       (net 3 GNDD))
     (pad 6 smd rect (at 0.65 0.2) (size 0.5 0.25) (layers F.Cu F.Paste F.Mask)
-      (net 271 "Net-(C78-Pad1)"))
+      (net 63 LMS_D3V3))
     (pad 7 smd rect (at 0.65 -0.2) (size 0.5 0.25) (layers F.Cu F.Paste F.Mask)
-      (net 271 "Net-(C78-Pad1)"))
+      (net 63 LMS_D3V3))
     (pad 8 smd rect (at 0.65 -0.6) (size 0.5 0.25) (layers F.Cu F.Paste F.Mask)
-      (net 271 "Net-(C78-Pad1)"))
+      (net 63 LMS_D3V3))
     (pad 9 smd rect (at 0 0) (size 0.35 1.4) (layers F.Cu F.Paste F.Mask)
       (net 3 GNDD))
@@
   )
   (module Capacitors_SMD:C_0603 (layer B.Cu)
-    (at 122.16 121.36 90)
+    (at 122.34 124.1 90)
     (descr "Capacitor SMD 0603, reflow soldering, AVX (see smccp.pdf)")
     (tags "capacitor 0603")
@@
     (fp_line (start 0.35 -0.6) (end -0.35 -0.6) (layer B.SilkS) (width 0.12))
     (pad 1 smd rect (at -0.75 0 90) (size 0.8 0.75) (layers B.Cu B.Paste B.Mask)
-      (net 271 "Net-(C78-Pad1)"))
+      (net 63 LMS_D3V3))
     (pad 2 smd rect (at 0.75 0 90) (size 0.8 0.75) (layers B.Cu B.Paste B.Mask)
       (net 3 GNDD))
@@
   )
   (module Capacitors_SMD:C_0603 (layer F.Cu)
-    (at 117.22 124.18 270)
+    (at 119.94 122.33)
     (descr "Capacitor SMD 0603, reflow soldering, AVX (see smccp.pdf)")
     (tags "capacitor 0603")
     (attr smd)
-    (fp_text reference C79 (at 0 -1.9 270) (layer F.SilkS)
+    (fp_text reference C79 (at 0 -1.9) (layer F.SilkS)
       (effects (font (size 1 1) (thickness 0.15)))
     )
-    (fp_text value 1u (at 0 1.9 270) (layer F.Fab)
+    (fp_text value 1u (at 0 1.9) (layer F.Fab)
       (effects (font (size 1 1) (thickness 0.15)))
     )
@@
     (fp_line (start -0.35 -0.6) (end 0.35 -0.6) (layer F.SilkS) (width 0.12))
     (fp_line (start 0.35 0.6) (end -0.35 0.6) (layer F.SilkS) (width 0.12))
-    (pad 1 smd rect (at -0.75 0 270) (size 0.8 0.75) (layers F.Cu F.Paste F.Mask)
+    (pad 1 smd rect (at -0.75 0) (size 0.8 0.75) (layers F.Cu F.Paste F.Mask)
       (net 247 "Net-(C79-Pad1)"))
-    (pad 2 smd rect (at 0.75 0 270) (size 0.8 0.75) (layers F.Cu F.Paste F.Mask)
+    (pad 2 smd rect (at 0.75 0) (size 0.8 0.75) (layers F.Cu F.Paste F.Mask)
       (net 3 GNDD))
     (model Capacitors_SMD.3dshapes/C_0603.wrl
@@
     )
   )
-  (module Capacitors_SMD:C_0805 (layer B.Cu)
-    (at 122.24 125.37 90)
+  (module Capacitors_SMD:C_0805 (layer F.Cu)
+    (at 117 124.05 270)
     (descr "Capacitor SMD 0805, reflow soldering, AVX (see smccp.pdf)")
     (tags "capacitor 0805")
     (attr smd)
-    (fp_text reference L3 (at 0 2.1 90) (layer B.SilkS)
-      (effects (font (size 1 1) (thickness 0.15)) (justify mirror))
+    (fp_text reference L3 (at 0 -2.1 270) (layer F.SilkS)
+      (effects (font (size 1 1) (thickness 0.15)))
     )
-    (fp_text value BLM18KG601SN1D (at 0 -2.1 90) (layer B.Fab)
-      (effects (font (size 1 1) (thickness 0.15)) (justify mirror))
+    (fp_text value BLM18KG601SN1D (at 0 2.1 270) (layer F.Fab)
+      (effects (font (size 1 1) (thickness 0.15)))
     )
-    (fp_line (start -1 -0.625) (end -1 0.625) (layer B.Fab) (width 0.1))
-    (fp_line (start 1 -0.625) (end -1 -0.625) (layer B.Fab) (width 0.1))
-    (fp_line (start 1 0.625) (end 1 -0.625) (layer B.Fab) (width 0.1))
-    (fp_line (start -1 0.625) (end 1 0.625) (layer B.Fab) (width 0.1))
-    (fp_line (start -1.8 1) (end 1.8 1) (layer B.CrtYd) (width 0.05))
-    (fp_line (start -1.8 -1) (end 1.8 -1) (layer B.CrtYd) (width 0.05))
-    (fp_line (start -1.8 1) (end -1.8 -1) (layer B.CrtYd) (width 0.05))
-    (fp_line (start 1.8 1) (end 1.8 -1) (layer B.CrtYd) (width 0.05))
-    (fp_line (start 0.5 0.85) (end -0.5 0.85) (layer B.SilkS) (width 0.12))
-    (fp_line (start -0.5 -0.85) (end 0.5 -0.85) (layer B.SilkS) (width 0.12))
-    (pad 1 smd rect (at -1 0 90) (size 1 1.25) (layers B.Cu B.Paste B.Mask)
-      (net 63 LMS_D3V3))
-    (pad 2 smd rect (at 1 0 90) (size 1 1.25) (layers B.Cu B.Paste B.Mask)
-      (net 271 "Net-(C78-Pad1)"))
+    (fp_line (start -1 0.625) (end -1 -0.625) (layer F.Fab) (width 0.1))
+    (fp_line (start 1 0.625) (end -1 0.625) (layer F.Fab) (width 0.1))
+    (fp_line (start 1 -0.625) (end 1 0.625) (layer F.Fab) (width 0.1))
+    (fp_line (start -1 -0.625) (end 1 -0.625) (layer F.Fab) (width 0.1))
+    (fp_line (start -1.8 -1) (end 1.8 -1) (layer F.CrtYd) (width 0.05))
+    (fp_line (start -1.8 1) (end 1.8 1) (layer F.CrtYd) (width 0.05))
+    (fp_line (start -1.8 -1) (end -1.8 1) (layer F.CrtYd) (width 0.05))
+    (fp_line (start 1.8 -1) (end 1.8 1) (layer F.CrtYd) (width 0.05))
+    (fp_line (start 0.5 -0.85) (end -0.5 -0.85) (layer F.SilkS) (width 0.12))
+    (fp_line (start -0.5 0.85) (end 0.5 0.85) (layer F.SilkS) (width 0.12))
+    (pad 1 smd rect (at -1 0 270) (size 1 1.25) (layers F.Cu F.Paste F.Mask)
+      (net 65 LMS_A3V3))
+    (pad 2 smd rect (at 1 0 270) (size 1 1.25) (layers F.Cu F.Paste F.Mask)
+      (net 247 "Net-(C79-Pad1)"))
     (model Capacitors_SMD.3dshapes/C_0805.wrl
       (at (xyz 0 0 0))
@@
   )
   (module Capacitors_SMD:C_0603 (layer F.Cu)
-    (at 102.53 132.49)
+    (at 79.89 132.73)
     (descr "Capacitor SMD 0603, reflow soldering, AVX (see smccp.pdf)")
     (tags "capacitor 0603")
@@
   )
   (module Capacitors_SMD:C_0603 (layer F.Cu)
-    (at 103.01 136.54)
+    (at 80.37 136.78)
     (descr "Capacitor SMD 0603, reflow soldering, AVX (see smccp.pdf)")
     (tags "capacitor 0603")
@@
   )
   (module Capacitors_SMD:C_0603 (layer F.Cu)
-    (at 102.29 140.58)
+    (at 79.65 140.82)
     (descr "Capacitor SMD 0603, reflow soldering, AVX (see smccp.pdf)")
     (tags "capacitor 0603")
@@
   )
   (module Capacitors_SMD:C_0603 (layer F.Cu)
-    (at 93.76 142.49)
+    (at 71.12 142.73)
     (descr "Capacitor SMD 0603, reflow soldering, AVX (see smccp.pdf)")
     (tags "capacitor 0603")
@@
   )
   (module Capacitors_SMD:C_0603 (layer F.Cu)
-    (at 98.25 143.42)
+    (at 75.61 143.66)
     (descr "Capacitor SMD 0603, reflow soldering, AVX (see smccp.pdf)")
     (tags "capacitor 0603")
@@
   )
   (module Resistors_SMD:R_0603 (layer F.Cu)
-    (at 98.25 139.75)
+    (at 75.1 139.53)
     (descr "Resistor SMD 0603, reflow soldering, Vishay (see dcrcw.pdf)")
     (tags "resistor 0603")
@@
   )
   (module Resistors_SMD:R_0603 (layer F.Cu)
-    (at 93.25 138.2)
+    (at 70.61 138.44)
     (descr "Resistor SMD 0603, reflow soldering, Vishay (see dcrcw.pdf)")
     (tags "resistor 0603")
@@
   )
   (module Resistors_SMD:R_0603 (layer F.Cu)
-    (at 97.77 136.3)
+    (at 75.13 136.54)
     (descr "Resistor SMD 0603, reflow soldering, Vishay (see dcrcw.pdf)")
     (tags "resistor 0603")
@@
   )
   (module Resistors_SMD:R_0603 (layer F.Cu)
-    (at 92.88 132.57)
+    (at 70.24 132.81)
     (descr "Resistor SMD 0603, reflow soldering, Vishay (see dcrcw.pdf)")
     (tags "resistor 0603")
@@
   )
   (module Resistors_SMD:R_0603 (layer F.Cu)
-    (at 97.81 132.85)
+    (at 75.17 133.09)
     (descr "Resistor SMD 0603, reflow soldering, Vishay (see dcrcw.pdf)")
     (tags "resistor 0603")
@@
   )
   (module Resistors_SMD:R_0603 (layer F.Cu)
-    (at 92.64 135.17)
+    (at 70 135.41)
     (descr "Resistor SMD 0603, reflow soldering, Vishay (see dcrcw.pdf)")
     (tags "resistor 0603")

Commit message: Full Rpi beginning
Parts:
- removed the REF** at (107.5, 126.6)
- added REF**: MountingHole_3.2mm_M3_DIN965_Pad, Mounting_Holes:MountingHole_3.2mm_M3_DIN965_Pad, F.Cu at (103.5, 152.5)
- added REF**: MountingHole_3.2mm_M3_DIN965_Pad, Mounting_Holes:MountingHole_3.2mm_M3_DIN965_Pad, F.Cu at (161.5, 152.5)
- moved C80 25.3 mm to (129.2, 152.8)
- moved C84 25.3 mm to (118.2, 138.0)
- moved C87 25.3 mm to (120.9, 134.5)
- moved C92 25.3 mm to (113.2, 133.5)
- moved C93 25.3 mm to (113.0, 143.5)
- moved L8 25.3 mm to (117.9, 146.6)
- moved R21 25.3 mm to (117.4, 140.8)
- moved T2 25.3 mm to (117.7, 133.5)
- moved U8 25.3 mm to (126.2, 153.1)
- moved C86 25.3 mm to (120.9, 132.4)
- moved C90 25.3 mm to (121.4, 146.6)
- moved C91 25.3 mm to (121.3, 148.9)
- moved C79 25.3 mm to (127.3, 146.5)
- moved C81 25.3 mm to (114.9, 137.8)
- moved L3 25.3 mm to (124.4, 148.2)
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Other:
- board size 65 x 30 mm -> 65 x 56 mm
Changed lines of the file:
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@@
     (links 696)
     (no_connects 271)
-    (area 99.924999 99.924999 165.075001 130.075001)
+    (area 99.924999 99.924999 165.075001 156.075001)
     (thickness 1.6)
-    (drawings 9)
+    (drawings 13)
     (tracks 1891)
     (zones 0)
-    (modules 161)
+    (modules 162)
     (nets 271)
   )
@@
     (add_net ~RPI_OE)
   )
+  (module Mounting_Holes:MountingHole_3.2mm_M3_DIN965_Pad locked (layer F.Cu)
+    (at 103.5 152.5)
+    (descr "Mounting Hole 3.2mm, M3, DIN965")
+    (tags "mounting hole 3.2mm m3 din965")
+    (fp_text reference REF** (at 0 -3.8) (layer F.SilkS) hide
+      (effects (font (size 1 1) (thickness 0.15)))
+    )
+    (fp_text value MountingHole_3.2mm_M3_DIN965_Pad (at 0 3.8) (layer F.Fab)
+      (effects (font (size 1 1) (thickness 0.15)))
+    )
+    (fp_circle (center 0 0) (end 2.8 0) (layer Cmts.User) (width 0.15))
+    (fp_circle (center 0 0) (end 3.05 0) (layer F.CrtYd) (width 0.05))
+    (pad 1 thru_hole circle (at 0 0) (size 5.6 5.6) (drill 3.2) (layers *.Cu *.Mask))
+  )
+  (module Mounting_Holes:MountingHole_3.2mm_M3_DIN965_Pad locked (layer F.Cu)
+    (at 161.5 152.5)
+    (descr "Mounting Hole 3.2mm, M3, DIN965")
+    (tags "mounting hole 3.2mm m3 din965")
+    (fp_text reference REF** (at 0 -3.8) (layer F.SilkS) hide
+      (effects (font (size 1 1) (thickness 0.15)))
+    )
+    (fp_text value MountingHole_3.2mm_M3_DIN965_Pad (at 0 3.8) (layer F.Fab)
+      (effects (font (size 1 1) (thickness 0.15)))
+    )
+    (fp_circle (center 0 0) (end 2.8 0) (layer Cmts.User) (width 0.15))
+    (fp_circle (center 0 0) (end 3.05 0) (layer F.CrtYd) (width 0.05))
+    (pad 1 thru_hole circle (at 0 0) (size 5.6 5.6) (drill 3.2) (layers *.Cu *.Mask))
+  )
   (module sdr-foots:DQFN-120_via_off_pad (layer F.Cu)
-    (at 120.9715 120.8 180)
+    (at 128.37306 144.99604 180)
     (solder_mask_margin 0.04826)
     (clearance 0.04826)
@@
   )
   (module sdr-foots:DFN-8-1EP_1.6x1.2mm_Pitch0.4mm (layer F.Cu)
-    (at 120.1 124.49)
+    (at 127.50156 148.68604)
     (descr "DC8 Package 8-Lead Plastic DFN (2mm x 2mm) (see Linear Technology DFN_8_05-08-1719.pdf)")
     (tags "DFN 0.4")
@@
   )
   (module sdr-foots:DFN-4 (layer F.Cu)
-    (at 118.81 128.92)
+    (at 126.21156 153.11604)
     (fp_text reference U8 (at 0.1 -1.6 180) (layer F.SilkS)
       (effects (font (size 1.2 1.2) (thickness 0.15)))
@@
   )
   (module sdr-foots:DFN-4 (layer F.Cu)
-    (at 109.04 113.87 90)
+    (at 116.44156 138.06604 90)
     (fp_text reference U9 (at 0.1 -1.6 270) (layer F.SilkS)
       (effects (font (size 1.2 1.2) (thickness 0.15)))
@@
   )
   (module Capacitors_SMD:C_0603 (layer F.Cu)
-    (at 119.94 122.33)
+    (at 127.34156 146.52604)
     (descr "Capacitor SMD 0603, reflow soldering, AVX (see smccp.pdf)")
     (tags "capacitor 0603")
@@
   )
   (module Capacitors_SMD:C_0603 (layer F.Cu)
-    (at 121.82 128.63)
+    (at 129.22156 152.82604)
     (descr "Capacitor SMD 0603, reflow soldering, AVX (see smccp.pdf)")
     (tags "capacitor 0603")
@@
   )
   (module Capacitors_SMD:C_0603 (layer B.Cu)
-    (at 107.49 113.61 270)
+    (at 114.89156 137.80604 270)
     (descr "Capacitor SMD 0603, reflow soldering, AVX (see smccp.pdf)")
     (tags "capacitor 0603")
@@
   )
   (module Capacitors_SMD:C_0603 (layer B.Cu)
-    (at 120.41 128.71)
+    (at 127.81156 152.90604)
     (descr "Capacitor SMD 0603, reflow soldering, AVX (see smccp.pdf)")
     (tags "capacitor 0603")
@@
   )
   (module Capacitors_SMD:C_0603 (layer F.Cu)
-    (at 110.84 113.84 90)
+    (at 118.24156 138.03604 90)
     (descr "Capacitor SMD 0603, reflow soldering, AVX (see smccp.pdf)")
     (tags "capacitor 0603")
@@
   )
   (module Resistors_SMD:R_0603 (layer F.Cu)
-    (at 109.83 111.14 180)
+    (at 117.23156 135.33604 180)
     (descr "Resistor SMD 0603, reflow soldering, Vishay (see dcrcw.pdf)")
     (tags "resistor 0603")
@@
   )
   (module Resistors_SMD:R_0603 (layer F.Cu)
-    (at 109.96 116.63)
+    (at 117.36156 140.82604)
     (descr "Resistor SMD 0603, reflow soldering, Vishay (see dcrcw.pdf)")
     (tags "resistor 0603")
@@
   )
   (module Capacitors_SMD:C_0805 (layer F.Cu)
-    (at 117 124.05 270)
+    (at 124.40156 148.24604 270)
     (descr "Capacitor SMD 0805, reflow soldering, AVX (see smccp.pdf)")
     (tags "capacitor 0805")
@@
   )
   (module Capacitors_SMD:C_0603 (layer F.Cu)
-    (at 113.51 108.19)
+    (at 120.91156 132.38604)
     (descr "Capacitor SMD 0603, reflow soldering, AVX (see smccp.pdf)")
     (tags "capacitor 0603")
@@
   )
   (module Capacitors_SMD:C_0603 (layer F.Cu)
-    (at 113.53 110.28)
+    (at 120.93156 134.47604)
     (descr "Capacitor SMD 0603, reflow soldering, AVX (see smccp.pdf)")
     (tags "capacitor 0603")
@@
   )
   (module Capacitors_SMD:C_0603 (layer F.Cu)
-    (at 113.98 122.41)
+    (at 121.38156 146.60604)
     (descr "Capacitor SMD 0603, reflow soldering, AVX (see smccp.pdf)")
     (tags "capacitor 0603")
@@
   )
   (module Capacitors_SMD:C_0603 (layer F.Cu)
-    (at 113.87 124.69)
+    (at 121.27156 148.88604)
     (descr "Capacitor SMD 0603, reflow soldering, AVX (see smccp.pdf)")
     (tags "capacitor 0603")
@@
   )
   (module sdr-foots:SMA_H (layer F.Cu)
-    (at 101.69 110.24792)
+    (at 101.69 133.68782)
     (attr smd)
     (fp_text reference J2 (at -0.05 -4.65) (layer F.SilkS) hide
@@
   )
   (module sdr-foots:SMA_H (layer F.Cu)
-    (at 102.7 119.89)
+    (at 102.7 145.14576)
     (attr smd)
     (fp_text reference J1 (at -0.05 -4.65) (layer F.SilkS) hide
@@
   )
   (module sdr-foots:B0322J5050 (layer F.Cu)
-    (at 108.9 119.92 90)
+    (at 116.30156 144.11604 90)
     (fp_text reference T1 (at -0.2 2.2 90) (layer F.SilkS)
       (effects (font (size 1 1) (thickness 0.15)))
@@
   )
   (module sdr-foots:B0322J5050 (layer F.Cu)
-    (at 110.34 109.35 180)
+    (at 117.74156 133.54604 180)
     (fp_text reference T2 (at -0.2 2.2 180) (layer F.SilkS)
       (effects (font (size 1 1) (thickness 0.15)))
@@
   )
   (module Capacitors_SMD:C_0603 (layer F.Cu)
-    (at 105.75 109.35 90)
+    (at 113.15156 133.54604 90)
     (descr "Capacitor SMD 0603, reflow soldering, AVX (see smccp.pdf)")
     (tags "capacitor 0603")
@@
   )
   (module Capacitors_SMD:C_0603 (layer F.Cu)
-    (at 105.56 119.32 90)
+    (at 112.96156 143.51604 90)
     (descr "Capacitor SMD 0603, reflow soldering, AVX (see smccp.pdf)")
     (tags "capacitor 0603")
@@
   )
   (module Inductors_SMD:L_0603 (layer F.Cu)
-    (at 117.11 108.17 180)
+    (at 124.51156 132.36604 180)
     (descr "Resistor SMD 0603, reflow soldering, Vishay (see dcrcw.pdf)")
     (tags "resistor 0603")
@@
   )
   (module Inductors_SMD:L_0603 (layer F.Cu)
-    (at 117.13 110.26 180)
+    (at 124.53156 134.45604 180)
     (descr "Resistor SMD 0603, reflow soldering, Vishay (see dcrcw.pdf)")
     (tags "resistor 0603")
@@
   )
   (module Inductors_SMD:L_0603 (layer F.Cu)
-    (at 110.49 122.41 180)
+    (at 117.89156 146.60604 180)
     (descr "Resistor SMD 0603, reflow soldering, Vishay (see dcrcw.pdf)")
     (tags "resistor 0603")
@@
   )
   (module Inductors_SMD:L_0603 (layer F.Cu)
-    (at 109.92 124.64 180)
+    (at 117.32156 148.83604 180)
     (descr "Resistor SMD 0603, reflow soldering, Vishay (see dcrcw.pdf)")
     (tags "resistor 0603")
@@
     )
   )
-  (module sdr-foots:shield (layer F.Cu)
-    (at 107.45 126.57)
-    (fp_text reference REF** (at 0 0.5) (layer F.SilkS) hide
-      (effects (font (size 1 1) (thickness 0.15)))
-    )
-    (fp_text value shield (at 0 -0.5) (layer F.Fab)
-      (effects (font (size 1 1) (thickness 0.15)))
-    )
-    (pad 1 smd rect (at 0 -3.25 90) (size 5.6 1) (layers F.Cu F.Paste F.Mask))
-    (pad 2 smd rect (at 0 -11.75 90) (size 5.6 1) (layers F.Cu F.Paste F.Mask))
-    (pad 3 smd rect (at 3.25 -20) (size 5.6 1) (layers F.Cu F.Paste F.Mask))
-    (pad 4 smd rect (at 15 -16.75 90) (size 5.6 1) (layers F.Cu F.Paste F.Mask))
-    (pad 5 smd rect (at 15 -3.25 90) (size 5.6 1) (layers F.Cu F.Paste F.Mask))
-    (pad 6 smd rect (at 7.5 0) (size 5.6 1) (layers F.Cu F.Paste F.Mask))
-  )
-  (gr_line (start 100 130) (end 100 100) (layer Edge.Cuts) (width 0.15))
-  (gr_line (start 165 130) (end 100 130) (layer Edge.Cuts) (width 0.15))
-  (gr_line (start 165 100) (end 165 130) (layer Edge.Cuts) (width 0.15))
-  (gr_line (start 100 100) (end 165 100) (layer Edge.Cuts) (width 0.15))
+  (gr_arc (start 103 153) (end 100 153) (angle -90) (layer Edge.Cuts) (width 0.15))
+  (gr_arc (start 162 153) (end 162 156) (angle -90) (layer Edge.Cuts) (width 0.15))
+  (gr_arc (start 162 103) (end 165 103) (angle -90) (layer Edge.Cuts) (width 0.15))
+  (gr_arc (start 103 103) (end 103 100) (angle -90) (layer Edge.Cuts) (width 0.15))
+  (gr_line (start 100 153) (end 100 103) (layer Edge.Cuts) (width 0.15))
+  (gr_line (start 162 156) (end 103 156) (layer Edge.Cuts) (width 0.15))
+  (gr_line (start 165 103) (end 165 153) (layer Edge.Cuts) (width 0.15))
+  (gr_line (start 103 100) (end 162 100) (layer Edge.Cuts) (width 0.15))
   (gr_line (start 158.1 106.3) (end 158.1 106.5) (angle 90) (layer F.CrtYd) (width 0.2))
   (gr_line (start 152.6 106.3) (end 158.1 106.3) (angle 90) (layer F.CrtYd) (width 0.2))
@@
     (polygon
       (pts
-        (xy 157.6 107) (xy 157.6 106) (xy 158.5 106) (xy 161.2 109) (xy 157.6 109)
-        (xy 157.6 107.3)
+        (xy 161.2 109) (xy 160.6 109) (xy 160.6 111.3) (xy 157.6 109) (xy 157.6 106)
+        (xy 158.5 106)
       )
     )
